Commit message: finished hand-eye-calib of franka and smarteye

File: franka_ros2_moveit2_ws/src/panda_description/urdf/panda.urdf (robot description, URDF)
Before this commit: robot panda, 12 links, 11 joints
Links:
- added link tcp
Joints:
- added joint tcp_joint: type fixed, parent panda_hand, child tcp, origin xyz=0 0 0.1122 rpy=0 0 0, axis 0 0 1
