Commit message: 1. update the latest config of franka urdf, srdf and driver 2. introduce moveit calibration for convenient hand-eye-calib

File: franka_ros1_control_ws/src/franka_ros/franka_description/robots/hand.xacro (robot description, xacro)
@@ -61,5 +61,5 @@
       <collision>
         <geometry>
-          <mesh filename="package://franka_description/meshes/visual/finger.stl"/>
+          <mesh filename="package://franka_description/meshes/collision/finger.stl"/>
         </geometry>
       </collision>
@@ -75,5 +75,5 @@
         <origin xyz="0 0 0" rpy="0 0 ${pi}"/>
         <geometry>
-          <mesh filename="package://franka_description/meshes/visual/finger.stl"/>
+          <mesh filename="package://franka_description/meshes/collision/finger.stl"/>
         </geometry>
       </collision>

File: franka_ros1_control_ws/src/franka_ros/franka_description/robots/panda_arm.xacro (robot description, xacro)
@@ -62,10 +62,10 @@
     </link>
     <joint name="${arm_id}_joint1" type="revolute">
-      <safety_controller k_position="100.0" k_velocity="40.0" soft_lower_limit="-2.8973" soft_upper_limit="2.8973"/>
+      <safety_controller k_position="100.0" k_velocity="40.0" soft_lower_limit="-2.8073" soft_upper_limit="2.8073"/>
       <origin rpy="0 0 0" xyz="0 0 0.333"/>
       <parent link="${arm_id}_link0"/>
       <child link="${arm_id}_link1"/>
       <axis xyz="0 0 1"/>
-      <limit effort="87" lower="-2.8973" upper="2.8973" velocity="2.1750"/>
+      <limit effort="87" lower="-2.8073" upper="2.8073" velocity="2.1750"/>
     </joint>
     <link name="${arm_id}_link2">
@@ -95,10 +95,10 @@
     </link>
     <joint name="${arm_id}_joint2" type="revolute">
-      <safety_controller k_position="100.0" k_velocity="40.0" soft_lower_limit="-1.7628" soft_upper_limit="1.7628"/>
+      <safety_controller k_position="100.0" k_velocity="40.0" soft_lower_limit="-1.7028" soft_upper_limit="1.7028"/>
       <origin rpy="${-pi/2} 0 0" xyz="0 0 0"/>
       <parent link="${arm_id}_link1"/>
       <child link="${arm_id}_link2"/>
       <axis xyz="0 0 1"/>
-      <limit effort="87" lower="-1.7628" upper="1.7628" velocity="2.1750"/>
+      <limit effort="87" lower="-1.7028" upper="1.7028" velocity="2.1750"/>
     </joint>
     <link name="${arm_id}_link3">
@@ -128,10 +128,10 @@
     </link>
     <joint name="${arm_id}_joint3" type="revolute">
-      <safety_controller k_position="100.0" k_velocity="40.0" soft_lower_limit="-2.8973" soft_upper_limit="2.8973"/>
+      <safety_controller k_position="100.0" k_velocity="40.0" soft_lower_limit="-2.8073" soft_upper_limit="2.8073"/>
       <origin rpy="${pi/2} 0 0" xyz="0 -0.316 0"/>
       <parent link="${arm_id}_link2"/>
       <child link="${arm_id}_link3"/>
       <axis xyz="0 0 1"/>
-      <limit effort="87" lower="-2.8973" upper="2.8973" velocity="2.1750"/>
+      <limit effort="87" lower="-2.8073" upper="2.8073" velocity="2.1750"/>
     </joint>
     <link name="${arm_id}_link4">
@@ -161,10 +161,10 @@
     </link>
     <joint name="${arm_id}_joint4" type="revolute">
-      <safety_controller k_position="100.0" k_velocity="40.0" soft_lower_limit="-3.0718" soft_upper_limit="-0.0698"/>
+      <safety_controller k_position="100.0" k_velocity="40.0" soft_lower_limit="-3.0018" soft_upper_limit="-0.1298"/>
       <origin rpy="${pi/2} 0 0" xyz="0.0825 0 0"/>
       <parent link="${arm_id}_link3"/>
       <child link="${arm_id}_link4"/>
       <axis xyz="0 0 1"/>
-      <limit effort="87" lower="-3.0718" upper="-0.0698" velocity="2.1750"/>
+      <limit effort="87" lower="-3.0018" upper="-0.1298" velocity="2.1750"/>
     </joint>
     <link name="${arm_id}_link5">
@@ -212,10 +212,10 @@
     </link>
     <joint name="${arm_id}_joint5" type="revolute">
-      <safety_controller k_position="100.0" k_velocity="40.0" soft_lower_limit="-2.8973" soft_upper_limit="2.8973"/>
+      <safety_controller k_position="100.0" k_velocity="40.0" soft_lower_limit="-2.8073" soft_upper_limit="2.8073"/>
       <origin rpy="${-pi/2} 0 0" xyz="-0.0825 0.384 0"/>
       <parent link="${arm_id}_link4"/>
       <child link="${arm_id}_link5"/>
       <axis xyz="0 0 1"/>
-      <limit effort="12" lower="-2.8973" upper="2.8973" velocity="2.6100"/>
+      <limit effort="12" lower="-2.8073" upper="2.8073" velocity="2.6100"/>
     </joint>
     <link name="${arm_id}_link6">
@@ -245,10 +245,10 @@
     </link>
     <joint name="${arm_id}_joint6" type="revolute">
-      <safety_controller k_position="100.0" k_velocity="40.0" soft_lower_limit="-0.0175" soft_upper_limit="3.7525"/>
+      <safety_controller k_position="100.0" k_velocity="40.0" soft_lower_limit="0.0775" soft_upper_limit="3.7025"/>
       <origin rpy="${pi/2} 0 0" xyz="0 0 0"/>
       <parent link="${arm_id}_link5"/>
       <child link="${arm_id}_link6"/>
       <axis xyz="0 0 1"/>
-      <limit effort="12" lower="-0.0175" upper="3.7525" velocity="2.6100"/>
+      <limit effort="12" lower="0.0775" upper="3.7025" velocity="2.6100"/>
     </joint>
     <link name="${arm_id}_link7">
@@ -278,10 +278,10 @@
     </link>
     <joint name="${arm_id}_joint7" type="revolute">
-      <safety_controller k_position="100.0" k_velocity="40.0" soft_lower_limit="-2.8973" soft_upper_limit="2.8973"/>
+      <safety_controller k_position="100.0" k_velocity="40.0" soft_lower_limit="-2.8073" soft_upper_limit="2.8073"/>
       <origin rpy="${pi/2} 0 0" xyz="0.088 0 0"/>
       <parent link="${arm_id}_link6"/>
       <child link="${arm_id}_link7"/>
       <axis xyz="0 0 1"/>
-      <limit effort="12" lower="-2.8973" upper="2.8973" velocity="2.6100"/>
+      <limit effort="12" lower="-2.8073" upper="2.8073" velocity="2.6100"/>
     </joint>
     <link name="${arm_id}_link8">
